Commit message: moved teady model

File: assets/objects/urdf/teady_bear.urdf (robot description, URDF)
Before this commit: robot teady_bear, 1 links, 0 joints
Links:
- link base: geometry collision mesh filename=meshes/teady_bear/teady_bear.obj scale=.01 .01 .01; visual mesh filename=meshes/teady_bear/teady_bear.obj scale=.01 .01 .01
