Commit message: fixed sizing

File: assets/objects/urdf/power_drill.urdf (robot description, URDF)
Before this commit: robot power_drill, 1 links, 0 joints
Links:
- link base: geometry collision mesh filename=meshes/power_drill/textured.obj size=0.5 0.5 0.5; visual mesh filename=meshes/power_drill/textured.obj size=0.5 0.5 0.5
