Commit message: renamed teady to teddy, sim_trifinger saves to nerf data format

File: assets/objects/urdf/teddy_bear.urdf (robot description, URDF)
Before this commit: robot teady_bear, 1 links, 0 joints
Links:
- link base: geometry collision mesh filename=meshes/teddy_bear/teddy_bear.obj scale=.01 .01 .01; visual mesh filename=meshes/teddy_bear/teddy_bear.obj scale=.01 .01 .01
