Commit message: working grasp dicing etc

File: assets/objects/urdf/cube_multicolor.urdf (robot description, URDF)
Before this commit: robot object, 1 links, 0 joints
Links:
- link object: geometry collision box size=0.075 0.075 0.075; visual mesh filename=meshes/cube_multicolor.obj scale=.075 .075 .075
