Commit message: added support for bleach bottle

File: assets/objects/urdf/bleach_cleanser.urdf (robot description, URDF)
Before this commit: robot bleach_cleanser, 1 links, 0 joints
Links:
- link base: geometry collision mesh filename=meshes/bleach_cleanser/textured.obj scale=0.75 0.75 0.75; visual mesh filename=meshes/bleach_cleanser/textured.obj scale=0.75 0.75 0.75
