Commit message: size wasn't working moved to scale urdf

File: assets/objects/urdf/banana.urdf (robot description, URDF)
Before this commit: robot banana, 1 links, 0 joints
Links:
- link base: geometry collision mesh filename=meshes/banana/textured.obj scale=1.0 1.0 1.0; visual mesh filename=meshes/banana/textured.obj scale=1.0 1.0 1.0

File: assets/objects/urdf/bleach_cleanser.urdf (robot description, URDF)
Before this commit: robot bleach_cleanser, 1 links, 0 joints
Links:
- link base: geometry collision mesh filename=meshes/bleach_cleanser/textured.obj scale=1.0 1.0 1.0; visual mesh filename=meshes/bleach_cleanser/textured.obj scale=1.0 1.0 1.0

File: assets/objects/urdf/mug.urdf (robot description, URDF)
Before this commit: robot mug, 1 links, 0 joints
Links:
- link base: geometry collision mesh filename=meshes/mug/textured.obj scale=1.0 1.0 1.0; visual mesh filename=meshes/mug/textured.obj scale=1.0 1.0 1.0

File: assets/objects/urdf/power_drill.urdf (robot description, URDF)
Before this commit: robot power_drill, 1 links, 0 joints
Links:
- link base: geometry collision mesh filename=meshes/power_drill/textured.obj scale=1.0 1.0 1.0; visual mesh filename=meshes/power_drill/textured.obj scale=1.0 1.0 1.0

File: assets/objects/urdf/spatula.urdf (robot description, URDF)
Before this commit: robot spatula, 1 links, 0 joints
Links:
- link base: geometry collision mesh filename=meshes/spatula/textured.obj scale=1.0 1.0 1.0; visual mesh filename=meshes/spatula/textured.obj scale=1.0 1.0 1.0

Commit message: (WIP) reorganized asset meshes + removed scaling; changed CEM covariance

File: assets/objects/urdf/banana.urdf (robot description, URDF)
Before this commit: robot banana, 1 links, 0 joints
Links:
- link base: geometry collision mesh filename=meshes/banana/textured.obj; visual mesh filename=meshes/banana/textured.obj

File: assets/objects/urdf/bleach_cleanser.urdf (robot description, URDF)
Before this commit: robot bleach_cleanser, 1 links, 0 joints
Links:
- link base: geometry collision mesh filename=meshes/bleach_cleanser/textured.obj; visual mesh filename=meshes/bleach_cleanser/textured.obj

File: assets/objects/urdf/mug.urdf (robot description, URDF)
Before this commit: robot mug, 1 links, 0 joints
Links:
- link base: geometry collision mesh filename=meshes/mug/textured.obj; visual mesh filename=meshes/mug/textured.obj

File: assets/objects/urdf/power_drill.urdf (robot description, URDF)
Before this commit: robot power_drill, 1 links, 0 joints
Links:
- link base: geometry collision mesh filename=meshes/power_drill/textured.obj; visual mesh filename=meshes/power_drill/textured.obj

File: assets/objects/urdf/spatula.urdf (robot description, URDF)
Before this commit: robot spatula, 1 links, 0 joints
Links:
- link base: geometry collision mesh filename=meshes/spatula/textured.obj; visual mesh filename=meshes/spatula/textured.obj

File: assets/objects/urdf/teddy_bear.urdf (robot description, URDF)
Before this commit: robot teddy_bear, 1 links, 0 joints
Links:
- link base: geometry collision mesh filename=meshes/teddy_bear/textured.obj; visual mesh filename=meshes/teddy_bear/textured.obj
