Commit message: Add in all acronym urdfs to ig_objects

File: assets/objects/urdf/Xbox360_14e5dba73b283dc7fe0939859a0b15ea.urdf (robot description, URDF)
Before this commit: robot Xbox360_14e5dba73b283dc7fe0939859a0b15ea, 1 links, 0 joints
Links:
- link base: geometry collision mesh filename=meshes/Xbox360/14e5dba73b283dc7fe0939859a0b15ea.obj scale=0.01 0.01 0.01; visual mesh filename=meshes/Xbox360/14e5dba73b283dc7fe0939859a0b15ea.obj scale=0.01 0.01 0.01
