Commit message: Change urdf density and scaling to match acronym

File: assets/objects/urdf/1Shelves_12a64182bbaee7a12b2444829a3507de.urdf (robot description, URDF)
Before this commit: robot 1Shelves_12a64182bbaee7a12b2444829a3507de, 1 links, 0 joints
Links:
- link base: geometry collision mesh filename=meshes/1Shelves/12a64182bbaee7a12b2444829a3507de.obj; visual mesh filename=meshes/1Shelves/12a64182bbaee7a12b2444829a3507de.obj

File: assets/objects/urdf/1Shelves_160684937ae737ec5057ad0f363d6ddd.urdf (robot description, URDF)
Before this commit: robot 1Shelves_160684937ae737ec5057ad0f363d6ddd, 1 links, 0 joints
Links:
- link base: geometry collision mesh filename=meshes/1Shelves/160684937ae737ec5057ad0f363d6ddd.obj; visual mesh filename=meshes/1Shelves/160684937ae737ec5057ad0f363d6ddd.obj

File: assets/objects/urdf/1Shelves_1e3df0ab57e8ca8587f357007f9e75d1.urdf (robot description, URDF)
Before this commit: robot 1Shelves_1e3df0ab57e8ca8587f357007f9e75d1, 1 links, 0 joints
Links:
- link base: geometry collision mesh filename=meshes/1Shelves/1e3df0ab57e8ca8587f357007f9e75d1.obj; visual mesh filename=meshes/1Shelves/1e3df0ab57e8ca8587f357007f9e75d1.obj

File: assets/objects/urdf/1Shelves_2b9d60c74bc0d18ad8eae9bce48bbeed.urdf (robot description, URDF)
Before this commit: robot 1Shelves_2b9d60c74bc0d18ad8eae9bce48bbeed, 1 links, 0 joints
Links:
- link base: geometry collision mesh filename=meshes/1Shelves/2b9d60c74bc0d18ad8eae9bce48bbeed.obj; visual mesh filename=meshes/1Shelves/2b9d60c74bc0d18ad8eae9bce48bbeed.obj

File: assets/objects/urdf/1Shelves_4075b78276e39db2f59ac8a5783023e7.urdf (robot description, URDF)
Before this commit: robot 1Shelves_4075b78276e39db2f59ac8a5783023e7, 1 links, 0 joints
Links:
- link base: geometry collision mesh filename=meshes/1Shelves/4075b78276e39db2f59ac8a5783023e7.obj; visual mesh filename=meshes/1Shelves/4075b78276e39db2f59ac8a5783023e7.obj

File: assets/objects/urdf/1Shelves_842be31d76d29df0a00888d2bacdd893.urdf (robot description, URDF)
Before this commit: robot 1Shelves_842be31d76d29df0a00888d2bacdd893, 1 links, 0 joints
Links:
- link base: geometry collision mesh filename=meshes/1Shelves/842be31d76d29df0a00888d2bacdd893.obj; visual mesh filename=meshes/1Shelves/842be31d76d29df0a00888d2bacdd893.obj

File: assets/objects/urdf/1Shelves_a9c2bcc286b68ee217a3b9ca1765e2a4.urdf (robot description, URDF)
Before this commit: robot 1Shelves_a9c2bcc286b68ee217a3b9ca1765e2a4, 1 links, 0 joints
Links:
- link base: geometry collision mesh filename=meshes/1Shelves/a9c2bcc286b68ee217a3b9ca1765e2a4.obj; visual mesh filename=meshes/1Shelves/a9c2bcc286b68ee217a3b9ca1765e2a4.obj

File: assets/objects/urdf/1Shelves_ba5bf7a8a14c27086f9e9f74beb7c348.urdf (robot description, URDF)
Before this commit: robot 1Shelves_ba5bf7a8a14c27086f9e9f74beb7c348, 1 links, 0 joints
Links:
- link base: geometry collision mesh filename=meshes/1Shelves/ba5bf7a8a14c27086f9e9f74beb7c348.obj; visual mesh filename=meshes/1Shelves/ba5bf7a8a14c27086f9e9f74beb7c348.obj

File: assets/objects/urdf/2Shelves_1ab8202a944a6ff1de650492e45fb14f.urdf (robot description, URDF)
Before this commit: robot 2Shelves_1ab8202a944a6ff1de650492e45fb14f, 1 links, 0 joints
Links:
- link base: geometry collision mesh filename=meshes/2Shelves/1ab8202a944a6ff1de650492e45fb14f.obj; visual mesh filename=meshes/2Shelves/1ab8202a944a6ff1de650492e45fb14f.obj

File: assets/objects/urdf/2Shelves_3eb855c7bda95c1391c352d02061b3f7.urdf (robot description, URDF)
Before this commit: robot 2Shelves_3eb855c7bda95c1391c352d02061b3f7, 1 links, 0 joints
Links:
- link base: geometry collision mesh filename=meshes/2Shelves/3eb855c7bda95c1391c352d02061b3f7.obj; visual mesh filename=meshes/2Shelves/3eb855c7bda95c1391c352d02061b3f7.obj

File: assets/objects/urdf/2Shelves_8bdeeb23612c91c098d5fc0473d00a1c.urdf (robot description, URDF)
Before this commit: robot 2Shelves_8bdeeb23612c91c098d5fc0473d00a1c, 1 links, 0 joints
Links:
- link base: geometry collision mesh filename=meshes/2Shelves/8bdeeb23612c91c098d5fc0473d00a1c.obj; visual mesh filename=meshes/2Shelves/8bdeeb23612c91c098d5fc0473d00a1c.obj

File: assets/objects/urdf/2Shelves_b6a8f5a11d86e695157c9a82222f42ea.urdf (robot description, URDF)
Before this commit: robot 2Shelves_b6a8f5a11d86e695157c9a82222f42ea, 1 links, 0 joints
Links:
- link base: geometry collision mesh filename=meshes/2Shelves/b6a8f5a11d86e695157c9a82222f42ea.obj; visual mesh filename=meshes/2Shelves/b6a8f5a11d86e695157c9a82222f42ea.obj

File: assets/objects/urdf/2Shelves_cb87ed53ab8d2a50f4af63522c219933.urdf (robot description, URDF)
Before this commit: robot 2Shelves_cb87ed53ab8d2a50f4af63522c219933, 1 links, 0 joints
Links:
- link base: geometry collision mesh filename=meshes/2Shelves/cb87ed53ab8d2a50f4af63522c219933.obj; visual mesh filename=meshes/2Shelves/cb87ed53ab8d2a50f4af63522c219933.obj

File: assets/objects/urdf/2Shelves_dca2cd661bece47bd810b14a81e12eca.urdf (robot description, URDF)
Before this commit: robot 2Shelves_dca2cd661bece47bd810b14a81e12eca, 1 links, 0 joints
Links:
- link base: geometry collision mesh filename=meshes/2Shelves/dca2cd661bece47bd810b14a81e12eca.obj; visual mesh filename=meshes/2Shelves/dca2cd661bece47bd810b14a81e12eca.obj

File: assets/objects/urdf/2Shelves_df03b94777b1f0f9e4e3c2d62691be9.urdf (robot description, URDF)
Before this commit: robot 2Shelves_df03b94777b1f0f9e4e3c2d62691be9, 1 links, 0 joints
Links:
- link base: geometry collision mesh filename=meshes/2Shelves/df03b94777b1f0f9e4e3c2d62691be9.obj; visual mesh filename=meshes/2Shelves/df03b94777b1f0f9e4e3c2d62691be9.obj

File: assets/objects/urdf/2Shelves_f61465baa4c1c36de6089046407cf8f2.urdf (robot description, URDF)
Before this commit: robot 2Shelves_f61465baa4c1c36de6089046407cf8f2, 1 links, 0 joints
Links:
- link base: geometry collision mesh filename=meshes/2Shelves/f61465baa4c1c36de6089046407cf8f2.obj; visual mesh filename=meshes/2Shelves/f61465baa4c1c36de6089046407cf8f2.obj

File: assets/objects/urdf/3Shelves_10eb10fe18126d45b97ad864945165a1.urdf (robot description, URDF)
Before this commit: robot 3Shelves_10eb10fe18126d45b97ad864945165a1, 1 links, 0 joints
Links:
- link base: geometry collision mesh filename=meshes/3Shelves/10eb10fe18126d45b97ad864945165a1.obj; visual mesh filename=meshes/3Shelves/10eb10fe18126d45b97ad864945165a1.obj

File: assets/objects/urdf/3Shelves_22fbb23ca13c345b51887beb710d662a.urdf (robot description, URDF)
Before this commit: robot 3Shelves_22fbb23ca13c345b51887beb710d662a, 1 links, 0 joints
Links:
- link base: geometry collision mesh filename=meshes/3Shelves/22fbb23ca13c345b51887beb710d662a.obj; visual mesh filename=meshes/3Shelves/22fbb23ca13c345b51887beb710d662a.obj

File: assets/objects/urdf/3Shelves_29b66fc9db2f1558e0e89fd83955713c.urdf (robot description, URDF)
Before this commit: robot 3Shelves_29b66fc9db2f1558e0e89fd83955713c, 1 links, 0 joints
Links:
- link base: geometry collision mesh filename=meshes/3Shelves/29b66fc9db2f1558e0e89fd83955713c.obj; visual mesh filename=meshes/3Shelves/29b66fc9db2f1558e0e89fd83955713c.obj

File: assets/objects/urdf/3Shelves_3a3015426ff544c46fb17e2962e0eb20.urdf (robot description, URDF)
Before this commit: robot 3Shelves_3a3015426ff544c46fb17e2962e0eb20, 1 links, 0 joints
Links:
- link base: geometry collision mesh filename=meshes/3Shelves/3a3015426ff544c46fb17e2962e0eb20.obj; visual mesh filename=meshes/3Shelves/3a3015426ff544c46fb17e2962e0eb20.obj
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